File: MB02A1/Prototyping_phase/MainBoard/conn_module.kicad_sch (KiCad schematic)
At the start: 0 parts

Commit message: Design update, production preparation.
Parts:
- added ADC.1, ADC.2, DAC.1, EXTI.1, EXTI.2, EXTI.3, PWM.1, PWM.2, PWM.3, PWR3V3.1, PWR3V3.2, PWR3V3.3, PWR5V.1, PWR5V.2, PWR5V.3: Conn_01x02_Pin, Connector_PinHeader_2.54mm:PinHeader_1x02_P2.54mm_Vertical, symbol Connector:Conn_01x02_Pin
- added DISPLAY1: Conn_01x14_Pin, Connector_PinHeader_2.54mm:PinHeader_1x14_P2.54mm_Vertical, symbol Connector:Conn_01x14_Pin
- added EXIO.1, EXIO.2: Conn_01x08_Pin, Connector_PinHeader_2.54mm:PinHeader_1x08_P2.54mm_Vertical, symbol Connector:Conn_01x08_Pin
- added I2C1.1, I2C1.2, I2C1.3, I2C1.4: Conn_01x04_Pin, Connector_PinHeader_2.54mm:PinHeader_1x04_P2.54mm_Vertical, symbol Connector:Conn_01x04_Pin
- added SPI2.1, SPI2.2: Conn_01x06_Pin, Connector_PinHeader_2.54mm:PinHeader_1x06_P2.54mm_Vertical, symbol Connector:Conn_01x06_Pin
- added U12: MCP23017_SO, Package_SO:SOIC-28W_7.5x17.9mm_P1.27mm, symbol Interface_Expansion:MCP23017_SO
Connections:
- new net: EXIO.2.1 (Pin_1), U12.21 (GPA0)
- new net: EXIO.2.2 (Pin_2), U12.22 (GPA1)
- new net: EXIO.2.3 (Pin_3), U12.23 (GPA2)
- new net: EXIO.2.4 (Pin_4), U12.24 (GPA3)
- new net: EXIO.2.5 (Pin_5), U12.25 (GPA4)
- new net: EXIO.2.6 (Pin_6), U12.26 (GPA5)
- new net: EXIO.2.7 (Pin_7), U12.27 (GPA6)
- new net: EXIO.2.8 (Pin_8), U12.28 (GPA7)
- new net: EXIO.1.1 (Pin_1), U12.1 (GPB0)
- new net: EXIO.1.2 (Pin_2), U12.2 (GPB1)
- new net: EXIO.1.3 (Pin_3), U12.3 (GPB2)
- new net: EXIO.1.4 (Pin_4), U12.4 (GPB3)
- new net: EXIO.1.5 (Pin_5), U12.5 (GPB4)
- new net: EXIO.1.6 (Pin_6), U12.6 (GPB5)
- new net: EXIO.1.7 (Pin_7), U12.7 (GPB6)
- new net: EXIO.1.8 (Pin_8), U12.8 (GPB7)
- new net 5V_REG: DISPLAY1.1 (Pin_1), I2C1.1.3 (Pin_3), I2C1.2.3 (Pin_3), I2C1.3.3 (Pin_3), I2C1.4.3 (Pin_3), PWR5V.1.1 (Pin_1), PWR5V.2.1 (Pin_1), PWR5V.3.1 (Pin_1), SPI2.1.5 (Pin_5), SPI2.2.5 (Pin_5)
- new net ADC1: ADC.1.1 (Pin_1)
- new net ADC2: ADC.2.1 (Pin_1)
- new net DAC_OUT: DAC.1.1 (Pin_1)
- new net DISPL_BNESS: DISPLAY1.8 (Pin_8)
- new net DISPL_CS: DISPLAY1.3 (Pin_3)
- new net DISPL_DC: DISPLAY1.5 (Pin_5)
- new net DISPL_MISO: DISPLAY1.13 (Pin_13), DISPLAY1.9 (Pin_9)
- new net DISPL_MOSI: DISPLAY1.12 (Pin_12), DISPLAY1.6 (Pin_6)
- new net DISPL_RST: DISPLAY1.4 (Pin_4)
- new net DISPL_SCK: DISPLAY1.10 (Pin_10), DISPLAY1.7 (Pin_7)
- new net DISPL_TCH_CS: DISPLAY1.11 (Pin_11)
- new net DISPL_TIRQ: DISPLAY1.14 (Pin_14)
- new net EXTI1: EXTI.1.1 (Pin_1)
- new net EXTI2: EXTI.2.1 (Pin_1)
- new net EXTI3: EXTI.3.1 (Pin_1)
- new net GND: ADC.1.2 (Pin_2), ADC.2.2 (Pin_2), DAC.1.2 (Pin_2), DISPLAY1.2 (Pin_2), EXTI.1.2 (Pin_2), EXTI.2.2 (Pin_2), EXTI.3.2 (Pin_2), I2C1.1.4 (Pin_4), I2C1.2.4 (Pin_4), I2C1.3.4 (Pin_4), I2C1.4.4 (Pin_4), PWM.1.2 (Pin_2), PWM.2.2 (Pin_2), PWM.3.2 (Pin_2), PWR3V3.1.2 (Pin_2), PWR3V3.2.2 (Pin_2), PWR3V3.3.2 (Pin_2), PWR5V.1.2 (Pin_2), PWR5V.2.2 (Pin_2), PWR5V.3.2 (Pin_2), SPI2.1.6 (Pin_6), SPI2.2.6 (Pin_6), U12.10 (VSS), U12.15 (A0)
- new net I2C1_SCL: I2C1.1.1 (Pin_1), I2C1.2.1 (Pin_1), I2C1.3.1 (Pin_1), I2C1.4.1 (Pin_1), U12.12 (SCK)
- new net I2C1_SDA: I2C1.1.2 (Pin_2), I2C1.2.2 (Pin_2), I2C1.3.2 (Pin_2), I2C1.4.2 (Pin_2), U12.13 (SDA)
- new net M3V3: PWR3V3.1.1 (Pin_1), PWR3V3.2.1 (Pin_1), PWR3V3.3.1 (Pin_1)
- new net M5V: U12.16 (A1), U12.17 (A2), U12.18 (~{RESET}), U12.9 (VDD)
- new net PWM1: PWM.1.1 (Pin_1)
- new net PWM2: PWM.2.1 (Pin_1)
- new net PWM3: PWM.3.1 (Pin_1)
- new net SPI2_CS0: SPI2.1.1 (Pin_1)
- new net SPI2_CS1: SPI2.2.1 (Pin_1)
- new net SPI2_MISO: SPI2.1.4 (Pin_4), SPI2.2.4 (Pin_4)
- new net SPI2_MOSI: SPI2.1.3 (Pin_3), SPI2.2.3 (Pin_3)
- new net SPI2_SCK: SPI2.1.2 (Pin_2), SPI2.2.2 (Pin_2)
