File: MB02A1/Prototyping_phase/MainBoard/mb02a1.kicad_sch (KiCad schematic)
At the start: 0 parts

Commit message: Design update, production preparation.
Other:
- sheet Memory Modul renamed Memory Module
Changed lines of the file:
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@@
 			(color 255 255 194 1.0000)
 		)
-		(property "Sheetname" "Memory Modul"
+		(property "Sheetname" "Memory Module"
 			(at 25.4 75.4884 0)
 			(effects
